Commit message: Camera orientied to the correct direction

File: urdf/wrv4/wrv4.urdf.xacro (robot description, xacro)
@@ -23,5 +23,5 @@
     <color rgba="1 1 0 1"/>
   </material>
-  <!-- LINKS -->
+  <!--LINKS-->
   <link name="base_footprint"/>
   <link name="base_link">
@@ -169,6 +169,6 @@
   </link>
   <link name="imu_link">
-  </link>
-<!--JOINTS-->
+    </link>
+  <!--JOINTS-->
   <joint name="base_joint" type="fixed">
     <origin rpy="0 0 0" xyz="0 0 0.0875"/>
@@ -206,5 +206,5 @@
   </joint>
   <joint name="camera_optical_joint" type="fixed">
-    <origin rpy="0 1.57 0" xyz="0.015 0 0"/>
+    <origin rpy="0 0 0" xyz="0.015 0 0"/>
     <parent link="camera_link"/>
     <child link="camera_color_link"/>
@@ -220,5 +220,4 @@
     <child link="imu_link"/>
   </joint>
-<!--GAZEBO-->
   <gazebo reference="base_link">
     <material>Gazebo/White</material>

File: urdf/wrv4/wrv4.xacro (robot description, xacro)
@@ -183,5 +183,5 @@
     </joint>
     <joint name="camera_optical_joint" type="fixed">
-        <origin xyz="0.015 0 0" rpy="0 1.57 0"/>
+        <origin xyz="0.015 0 0" rpy="0 0 0"/>
         <parent link="camera_link"/>
         <child link="camera_color_link"/>
