Commit message: 1. Some changes to RViz2 config file.

File: urdf/wrv3/wrv3.xacro (robot description, xacro)
@@ -39,5 +39,5 @@
         <origin xyz="0 0 0" rpy="0 0 0"/>
         <mass value="0.303"/>
-        <inertia ixx="2.05e-04" iyy="2.05e-04" izz="7.58e-04" ixy="0" ixz="0" iyz="0"/>
+        <inertia ixx="2.05e-04" iyy="2.05e-04" izz="3.79e-04" ixy="0" ixz="0" iyz="0"/>
     </inertial>
     <visual>
@@ -65,5 +65,5 @@
         <origin xyz="0 0 0" rpy="0 0 0"/>
         <mass value="0.303"/>
-        <inertia ixx="2.05e-04" iyy="2.05e-04" izz="7.58e-04" ixy="0" ixz="0" iyz="0"/>
+        <inertia ixx="2.05e-04" iyy="2.05e-04" izz="3.79e-04" ixy="0" ixz="0" iyz="0"/>
     </inertial>
     <visual>
@@ -91,5 +91,5 @@
         <origin xyz="0 0 0" rpy="0 0 0"/>
         <mass value="0.303"/>
-        <inertia ixx="2.05e-04" iyy="2.05e-04" izz="7.58e-04" ixy="0" ixz="0" iyz="0"/>
+        <inertia ixx="2.05e-04" iyy="2.05e-04" izz="3.79e-04" ixy="0" ixz="0" iyz="0"/>
     </inertial>
     <visual>
@@ -117,5 +117,5 @@
         <origin xyz="0 0 0" rpy="0 0 0"/>
         <mass value="0.303"/>
-        <inertia ixx="2.05e-04" iyy="2.05e-04" izz="7.58e-04" ixy="0" ixz="0" iyz="0"/>
+        <inertia ixx="2.05e-04" iyy="2.05e-04" izz="3.79e-04" ixy="0" ixz="0" iyz="0"/>
     </inertial>
     <visual>

Commit message: Some minimal changes in the launch file

File: urdf/wrv3/wrv3.xacro (robot description, xacro)
@@ -56,5 +56,5 @@
 </link>
 <joint name="wheelr_joint" type="continuous">
-    <origin xyz="-0.1 -0.1125 0.05" rpy="-1.571 0 0"/>
+    <origin xyz="-0.1 -0.1125 0.05" rpy="1.571 0 0"/>
     <parent link="base_link"/>
     <child link="wheelr_link"/>
@@ -82,5 +82,5 @@
 </link>
 <joint name="wheeldl_joint" type="continuous">
-    <origin xyz="0.1 0.1125 0.05" rpy="1.571 0 0"/>
+    <origin xyz="0.1 0.1125 0.05" rpy="-1.571 0 0"/>
     <parent link="base_link"/>
     <child link="wheeldl_link"/>
