Commit message: The robot is finally moving, but can't take turns.

File: urdf/wrv3/materials.xacro (robot description, xacro)
@@ -10,4 +10,7 @@
   <color rgba="1 0 0 1"/>
 </material>
+<material name="yellow">
+  <color rgba="1 1 0 1"/>
+</material>
 <material name="blue">
   <color rgba="0 0 1 1"/>

File: urdf/wrv3/wrv3.xacro (robot description, xacro)
@@ -30,5 +30,5 @@
 </link>
 <joint name="wheell_joint" type="continuous">
-    <origin xyz="-0.1 0.1125 0.05" rpy="1.571 0 0"/>
+    <origin xyz="-0.1 0.1125 0.05" rpy="-1.571 0 0"/>
     <parent link="base_link"/>
     <child link="wheell_link"/>
@@ -46,5 +46,5 @@
             <mesh filename="package://robot_launcher_cpp/meshes/wheel.stl" scale="0.01 0.01 0.01"/>
         </geometry>
-        <material name="red"/>
+        <material name="yellow"/>
     </visual>
     <collision>
@@ -72,5 +72,5 @@
             <mesh filename="package://robot_launcher_cpp/meshes/wheel.stl" scale="0.01 0.01 0.01"/>
         </geometry>
-        <material name="red"/>
+        <material name="yellow"/>
     </visual>
     <collision>
@@ -82,5 +82,5 @@
 </link>
 <joint name="wheeldl_joint" type="continuous">
-    <origin xyz="0.1 0.1125 0.05" rpy="1.571 0 0"/>
+    <origin xyz="0.1 0.1125 0.05" rpy="-1.571 0 0"/>
     <parent link="base_link"/>
     <child link="wheeldl_link"/>
@@ -142,5 +142,5 @@
         <origin xyz="0 0 0" rpy="0 0 0"/>
         <mass value="0.116"/>
-        <inertia ixx="1.47e-05" iyy="1.03e-04" izz="1.05e-04" ixy="0" ixz="0" iyz="0"/>
+        <inertia ixx="1.03e-04" iyy="1.47e-05" izz="1.05e-04" ixy="0" ixz="0" iyz="0"/>
     </inertial>
     <visual>
@@ -173,5 +173,5 @@
         <origin xyz="0 0 0" rpy="0 0 0"/>
         <mass value="0.232"/>
-        <inertia ixx="1.1e-04" iyy="1.1e-04" izz="3.09e-05" ixy="0" ixz="0" iyz="0"/>
+        <inertia ixx="1.102e-04" iyy="1.102e-04" izz="1.856e-04" ixy="0" ixz="0" iyz="0"/>
     </inertial>
     <visual>

Commit message: Now the robot file works with stl files for geometry.

File: urdf/wrv3/materials.xacro (robot description, xacro)
@@ -1,4 +1,4 @@
 <?xml version="1.0" ?>
-<robot name="wrv3" xmlns:xacro="http://www.ros.org/wiki/xacro" >
+<robot name="wrv4" xmlns:xacro="http://www.ros.org/wiki/xacro" >
 <material name="pet">
   <color rgba="0.700 0.700 0.700 1.000"/>
@@ -16,3 +16,6 @@
   <color rgba="1 1 1 1"/>
 </material>
+<material name="yellow">
+  <color rgba="1 1 0 1"/>
+</material>
 </robot>

File: urdf/wrv3/wrv3.urdf.xacro (robot description, xacro)
@@ -20,212 +20,220 @@
     <color rgba="1 1 1 1"/>
   </material>
+  <material name="yellow">
+    <color rgba="1 1 0 1"/>
+  </material>
+  <!--LINKS-->
   <link name="base_footprint"/>
+  <link name="base_link">
+    <inertial>
+      <origin rpy="0 0 0" xyz="0 0 0.0"/>
+      <mass value="6.935"/>
+      <inertia ixx="0.026" ixy="0" ixz="0" iyy="0.055" iyz="0" izz="0.075"/>
+    </inertial>
+    <visual>
+      <origin rpy="0 0 0" xyz="0 0 0.0"/>
+      <geometry>
+        <mesh filename="package://robot_launcher_cpp/meshes/base_link.stl" scale="0.01 0.01 0.01"/>
+      </geometry>
+      <material name="white"/>
+    </visual>
+    <collision>
+      <origin rpy="0 0 0" xyz="0 0 0.0"/>
+      <geometry>
+        <mesh filename="package://robot_launcher_cpp/meshes/base_link.stl" scale="0.01 0.01 0.01"/>
+      </geometry>
+    </collision>
+  </link>
+  <link name="wheelfl_link">
+    <inertial>
+      <origin rpy="0 0 0" xyz="0 0 0"/>
+      <mass value="0.303"/>
+      <inertia ixx="2.05e-04" ixy="0" ixz="0" iyy="2.05e-04" iyz="0" izz="3.79e-04"/>
+    </inertial>
+    <visual>
+      <origin rpy="0 0 0" xyz="0 0 0"/>
+      <geometry>
+        <mesh filename="package://robot_launcher_cpp/meshes/wheel.stl" scale="0.01 0.01 0.01"/>
+      </geometry>
+      <material name="red"/>
+    </visual>
+    <collision>
+      <origin rpy="0 0 0" xyz="0 0 0"/>
+      <geometry>
+        <mesh filename="package://robot_launcher_cpp/meshes/wheel.stl" scale="0.01 0.01 0.01"/>
+      </geometry>
+    </collision>
+  </link>
+  <link name="wheelfr_link">
+    <inertial>
+      <origin rpy="0 0 0" xyz="0 0 0"/>
+      <mass value="0.303"/>
+      <inertia ixx="2.05e-04" ixy="0" ixz="0" iyy="2.05e-04" iyz="0" izz="3.79e-04"/>
+    </inertial>
+    <visual>
+      <origin rpy="0 0 0" xyz="0 0 0"/>
+      <geometry>
+        <mesh filename="package://robot_launcher_cpp/meshes/wheel.stl" scale="0.01 0.01 0.01"/>
+      </geometry>
+      <material name="red"/>
+    </visual>
+    <collision>
+      <origin rpy="0 0 0" xyz="0 0 0"/>
+      <geometry>
+        <mesh filename="package://robot_launcher_cpp/meshes/wheel.stl" scale="0.01 0.01 0.01"/>
+      </geometry>
+    </collision>
+  </link>
+  <link name="wheelbl_link">
+    <inertial>
+      <origin rpy="0 0 0" xyz="0 0 0"/>
+      <mass value="0.303"/>
+      <inertia ixx="2.05e-04" ixy="0" ixz="0" iyy="2.05e-04" iyz="0" izz="3.79e-04"/>
+    </inertial>
+    <visual>
+      <origin rpy="0 0 0" xyz="0 0 0"/>
+      <geometry>
+        <mesh filename="package://robot_launcher_cpp/meshes/wheel.stl" scale="0.01 0.01 0.01"/>
+      </geometry>
+      <material name="yellow"/>
+    </visual>
+    <collision>
+      <origin rpy="0 0 0" xyz="0 0 0"/>
+      <geometry>
+        <mesh filename="package://robot_launcher_cpp/meshes/wheel.stl" scale="0.01 0.01 0.01"/>
+      </geometry>
+    </collision>
+  </link>
+  <link name="wheelbr_link">
+    <inertial>
+      <origin rpy="0 0 0" xyz="0 0 0"/>
+      <mass value="0.303"/>
+      <inertia ixx="2.05e-04" ixy="0" ixz="0" iyy="2.05e-04" iyz="0" izz="3.79e-04"/>
+    </inertial>
+    <visual>
+      <origin rpy="0 0 0" xyz="0 0 0"/>
+      <geometry>
+        <mesh filename="package://robot_launcher_cpp/meshes/wheel.stl" scale="0.01 0.01 0.01"/>
+      </geometry>
+      <material name="yellow"/>
+    </visual>
+    <collision>
+      <origin rpy="0 0 0" xyz="0 0 0"/>
+      <geometry>
+        <mesh filename="package://robot_launcher_cpp/meshes/wheel.stl" scale="0.01 0.01 0.01"/>
+      </geometry>
+    </collision>
+  </link>
+  <link name="camera_link">
+    <inertial>
+      <origin rpy="0 0 0" xyz="0 0 0"/>
+      <mass value="0.116"/>
+      <inertia ixx="1.03e-04" ixy="0" ixz="0" iyy="1.47e-05" iyz="0" izz="1.05e-04"/>
+    </inertial>
+    <visual>
+      <origin rpy="0 0 0" xyz="0 0 0"/>
+      <geometry>
+        <mesh filename="package://robot_launcher_cpp/meshes/camera.stl" scale="0.01 0.01 0.01"/>
+      </geometry>
+      <material name="blue"/>
+    </visual>
+    <collision>
+      <origin rpy="0 0 0" xyz="0 0 0"/>
+      <geometry>
+        <mesh filename="package://robot_launcher_cpp/meshes/camera.stl" scale="0.01 0.01 0.01"/>
+      </geometry>
+    </collision>
+  </link>
+  <link name="camera_color_link"/>
+  <link name="base_scan">
+    <inertial>
+      <origin rpy="0 0 0" xyz="0 0 0"/>
+      <mass value="0.232"/>
+      <inertia ixx="1.102e-04" ixy="0" ixz="0" iyy="1.102e-04" iyz="0" izz="1.856e-04"/>
+    </inertial>
+    <visual>
+      <origin rpy="0 0 0" xyz="0 0 0"/>
+      <geometry>
+        <mesh filename="package://robot_launcher_cpp/meshes/lidar.stl" scale="0.01 0.01 0.01"/>
+      </geometry>
+      <material name="green"/>
+    </visual>
+    <collision>
+      <origin rpy="0 0 0" xyz="0 0 0"/>
+      <geometry>
+        <mesh filename="package://robot_launcher_cpp/meshes/lidar.stl" scale="0.01 0.01 0.01"/>
+      </geometry>
+    </collision>
+  </link>
+  <link name="imu_link">
+    </link>
+  <!--JOINTS-->
   <joint name="base_joint" type="fixed">
-    <origin rpy="0 0 0" xyz="0 0 0.0"/>
+    <origin rpy="0 0 0" xyz="0 0 0.0875"/>
     <parent link="base_footprint"/>
     <child link="base_link"/>
+  </joint>
+  <joint name="wheelfl_joint" type="continuous">
+    <origin rpy="-1.571 0 0" xyz="0.1 0.1125 -0.0375"/>
+    <parent link="base_link"/>
+    <child link="wheelfl_link"/>
     <axis xyz="0 0 1"/>
   </joint>
-  <link name="base_link">
-    <inertial>
-      <origin rpy="0 0 0" xyz="0 0 0.0875"/>
-      <mass value="6.935"/>
-      <inertia ixx="0.026" ixy="0" ixz="0" iyy="0.055" iyz="0" izz="0.075"/>
-    </inertial>
-    <visual>
-      <origin rpy="0 0 0" xyz="0 0 0.0875"/>
-      <geometry>
-        <mesh filename="package://robot_launcher_cpp/meshes/base_link.stl" scale="0.01 0.01 0.01"/>
-      </geometry>
-      <material name="white"/>
-    </visual>
-    <collision>
-      <origin rpy="0 0 0" xyz="0 0 0.0875"/>
-      <geometry>
-        <mesh filename="package://robot_launcher_cpp/meshes/base_link.stl" scale="0.01 0.01 0.01"/>
-      </geometry>
-    </collision>
-  </link>
-  <joint name="wheell_joint" type="continuous">
-    <origin rpy="1.571 0 0" xyz="-0.1 0.1125 0.05"/>
-    <parent link="base_link"/>
-    <child link="wheell_link"/>
+  <joint name="wheelfr_joint" type="continuous">
+    <origin rpy="-1.571 0 0" xyz="0.1 -0.1125 -0.0375"/>
+    <parent link="base_link"/>
+    <child link="wheelfr_link"/>
     <axis xyz="0 0 1"/>
   </joint>
-  <link name="wheell_link">
-    <inertial>
-      <origin rpy="0 0 0" xyz="0 0 0"/>
-      <mass value="0.303"/>
-      <inertia ixx="2.05e-04" ixy="0" ixz="0" iyy="2.05e-04" iyz="0" izz="7.58e-04"/>
-    </inertial>
-    <visual>
-      <origin rpy="0 0 0" xyz="0 0 0"/>
-      <geometry>
-        <mesh filename="package://robot_launcher_cpp/meshes/wheel.stl" scale="0.01 0.01 0.01"/>
-      </geometry>
-      <material name="red"/>
-    </visual>
-    <collision>
-      <origin rpy="0 0 0" xyz="0 0 0"/>
-      <geometry>
-        <mesh filename="package://robot_launcher_cpp/meshes/wheel.stl" scale="0.01 0.01 0.01"/>
-      </geometry>
-    </collision>
-  </link>
-  <joint name="wheelr_joint" type="continuous">
-    <origin rpy="1.571 0 0" xyz="-0.1 -0.1125 0.05"/>
-    <parent link="base_link"/>
-    <child link="wheelr_link"/>
+  <joint name="wheelbl_joint" type="continuous">
+    <origin rpy="1.571 0 0" xyz="-0.1 0.1125 -0.0375"/>
+    <parent link="base_link"/>
+    <child link="wheelbl_link"/>
     <axis xyz="0 0 1"/>
   </joint>
-  <link name="wheelr_link">
-    <inertial>
-      <origin rpy="0 0 0" xyz="0 0 0"/>
-      <mass value="0.303"/>
-      <inertia ixx="2.05e-04" ixy="0" ixz="0" iyy="2.05e-04" iyz="0" izz="7.58e-04"/>
-    </inertial>
-    <visual>
-      <origin rpy="0 0 0" xyz="0 0 0"/>
-      <geometry>
-        <mesh filename="package://robot_launcher_cpp/meshes/wheel.stl" scale="0.01 0.01 0.01"/>
-      </geometry>
-      <material name="red"/>
-    </visual>
-    <collision>
-      <origin rpy="0 0 0" xyz="0 0 0"/>
-      <geometry>
-        <mesh filename="package://robot_launcher_cpp/meshes/wheel.stl" scale="0.01 0.01 0.01"/>
-      </geometry>
-    </collision>
-  </link>
-  <joint name="wheeldl_joint" type="continuous">
-    <origin rpy="-1.571 0 0" xyz="0.1 0.1125 0.05"/>
-    <parent link="base_link"/>
-    <child link="wheeldl_link"/>
+  <joint name="wheelbr_joint" type="continuous">
+    <origin rpy="1.571 0 0" xyz="-0.1 -0.1125 -0.0375"/>
+    <parent link="base_link"/>
+    <child link="wheelbr_link"/>
     <axis xyz="0 0 1"/>
   </joint>
-  <link name="wheeldl_link">
-    <inertial>
-      <origin rpy="0 0 0" xyz="0 0 0"/>
-      <mass value="0.303"/>
-      <inertia ixx="2.05e-04" ixy="0" ixz="0" iyy="2.05e-04" iyz="0" izz="7.58e-04"/>
-    </inertial>
-    <visual>
-      <origin rpy="0 0 0" xyz="0 0 0"/>
-      <geometry>
-        <mesh filename="package://robot_launcher_cpp/meshes/wheel.stl" scale="0.01 0.01 0.01"/>
-      </geometry>
-      <material name="red"/>
-    </visual>
-    <collision>
-      <origin rpy="0 0 0" xyz="0 0 0"/>
-      <geometry>
-        <mesh filename="package://robot_launcher_cpp/meshes/wheel.stl" scale="0.01 0.01 0.01"/>
-      </geometry>
-    </collision>
-  </link>
-  <joint name="wheeldr_joint" type="continuous">
-    <origin rpy="-1.571 0 0" xyz="0.1 -0.1125 0.05"/>
-    <parent link="base_link"/>
-    <child link="wheeldr_link"/>
-    <axis xyz="0 0 1"/>
-  </joint>
-  <link name="wheeldr_link">
-    <inertial>
-      <origin rpy="0 0 0" xyz="0 0 0"/>
-      <mass value="0.303"/>
-      <inertia ixx="2.05e-04" ixy="0" ixz="0" iyy="2.05e-04" iyz="0" izz="7.58e-04"/>
-    </inertial>
-    <visual>
-      <origin rpy="0 0 0" xyz="0 0 0"/>
-      <geometry>
-        <mesh filename="package://robot_launcher_cpp/meshes/wheel.stl" scale="0.01 0.01 0.01"/>
-      </geometry>
-      <material name="red"/>
-    </visual>
-    <collision>
-      <origin rpy="0 0 0" xyz="0 0 0"/>
-      <geometry>
-        <mesh filename="package://robot_launcher_cpp/meshes/wheel.stl" scale="0.01 0.01 0.01"/>
-      </geometry>
-    </collision>
-  </link>
   <joint name="camera_joint" type="fixed">
-    <origin rpy="0 0 0" xyz="0.165 0 0.0875"/>
+    <origin rpy="0 0 0" xyz="0.165 0 0.0"/>
     <parent link="base_link"/>
     <child link="camera_link"/>
   </joint>
-  <link name="camera_link">
-    <inertial>
-      <origin rpy="0 0 0" xyz="0 0 0"/>
-      <mass value="0.116"/>
-      <inertia ixx="1.47e-05" ixy="0" ixz="0" iyy="1.03e-04" iyz="0" izz="1.05e-04"/>
-    </inertial>
-    <visual>
-      <origin rpy="0 0 0" xyz="0 0 0"/>
-      <geometry>
-        <mesh filename="package://robot_launcher_cpp/meshes/camera.stl" scale="0.01 0.01 0.01"/>
-      </geometry>
-      <material name="blue"/>
-    </visual>
-    <collision>
-      <origin rpy="0 0 0" xyz="0 0 0"/>
-      <geometry>
-        <mesh filename="package://robot_launcher_cpp/meshes/camera.stl" scale="0.01 0.01 0.01"/>
-      </geometry>
-    </collision>
-  </link>
   <joint name="camera_optical_joint" type="fixed">
-    <origin rpy="0 1.57 0" xyz="0.015 0 0"/>
+    <origin rpy="0 0 0" xyz="0.015 0 0"/>
     <parent link="camera_link"/>
     <child link="camera_color_link"/>
   </joint>
-  <link name="camera_color_link"/>
   <joint name="lidar_joint" type="fixed">
-    <origin rpy="0 0 0" xyz="0.1 0 0.14"/>
+    <origin rpy="0 0 0" xyz="0.1 0 0.0525"/>
     <parent link="base_link"/>
     <child link="base_scan"/>
   </joint>
-  <link name="base_scan">
-    <inertial>
-      <origin rpy="0 0 0" xyz="0 0 0"/>
-      <mass value="0.232"/>
-      <inertia ixx="1.1e-04" ixy="0" ixz="0" iyy="1.1e-04" iyz="0" izz="3.09e-05"/>
-    </inertial>
-    <visual>
-      <origin rpy="0 0 0" xyz="0 0 0"/>
-      <geometry>
-        <mesh filename="package://robot_launcher_cpp/meshes/lidar.stl" scale="0.01 0.01 0.01"/>
-      </geometry>
-      <material name="green"/>
-    </visual>
-    <collision>
-      <origin rpy="0 0 0" xyz="0 0 0"/>
-      <geometry>
-        <mesh filename="package://robot_launcher_cpp/meshes/lidar.stl" scale="0.01 0.01 0.01"/>
-      </geometry>
-    </collision>
-  </link>
   <joint name="imu_joint" type="fixed">
-    <origin rpy="0 0 0" xyz="0 0 0.0875"/>
+    <origin rpy="0 0 0" xyz="0 0 0.0"/>
     <parent link="base_link"/>
     <child link="imu_link"/>
   </joint>
-  <link name="imu_link">
-</link>
   <gazebo reference="base_link">
     <material>Gazebo/White</material>
   </gazebo>
-  <gazebo reference="wheell_link">
+  <gazebo reference="wheelfl_link">
     <material>Gazebo/Red</material>
   </gazebo>
-  <gazebo reference="wheelr_link">
+  <gazebo reference="wheelfr_link">
     <material>Gazebo/Red</material>
   </gazebo>
-  <gazebo reference="wheeldl_link">
-    <material>Gazebo/Red</material>
-  </gazebo>
-  <gazebo reference="wheeldr_link">
-    <material>Gazebo/Red</material>
+  <gazebo reference="wheelbl_link">
+    <material>Gazebo/Yellow</material>
+    <mu1 value="0.0"/>
+    <mu2 value="0.0"/>
+  </gazebo>
+  <gazebo reference="wheelbr_link">
+    <material>Gazebo/Yellow</material>
+    <mu1 value="0.0"/>
+    <mu2 value="0.0"/>
   </gazebo>
   <gazebo reference="camera_link">
@@ -276,6 +284,6 @@
         </scan>
         <range>
-          <min>0.120000</min>
-          <max>3.5</max>
+          <min>0.12</min>
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