Commit message: Now the robot file works with stl files for geometry.

File: urdf/wrv3/wrv3.xacro (robot description, xacro)
@@ -1,199 +1,200 @@
 <?xml version="1.0"?>
 <robot name="wrv3" xmlns:xacro="http://www.ros.org/wiki/xacro">
-<xacro:include filename="materials.xacro"/>
-<link name="base_footprint"/>
-<joint name="base_joint" type="fixed">
-    <origin xyz="0 0 0.0" rpy="0 0 0"/>
-    <parent link="base_footprint"/>
-    <child link="base_link"/>
-    <axis xyz="0 0 1"/>
-</joint>
-<link name="base_link">
-    <inertial>
+    <xacro:include filename="materials.xacro"/>
+    <!--LINKS-->
+    <link name="base_footprint"/>
+    <link name="base_link">
+        <inertial>
+            <origin xyz="0 0 0.0" rpy="0 0 0"/>
+            <mass value="6.935"/>
+            <inertia ixx="0.026" iyy="0.055" izz="0.075" ixy="0" ixz="0" iyz="0"/>
+        </inertial>
+        <visual>
+            <origin xyz="0 0 0.0" rpy="0 0 0"/>
+            <geometry>
+                <mesh filename="package://robot_launcher_cpp/meshes/base_link.stl" scale="0.01 0.01 0.01"/>
+            </geometry>
+            <material name="white"/>
+        </visual>
+        <collision>
+            <origin xyz="0 0 0.0" rpy="0 0 0"/>
+            <geometry>
+                <mesh filename="package://robot_launcher_cpp/meshes/base_link.stl" scale="0.01 0.01 0.01"/>
+            </geometry>
+        </collision>
+    </link>
+    <link name="wheelfl_link">
+        <inertial>
+            <origin xyz="0 0 0" rpy="0 0 0"/>
+            <mass value="0.303"/>
+            <inertia ixx="2.05e-04" iyy="2.05e-04" izz="3.79e-04" ixy="0" ixz="0" iyz="0"/>
+        </inertial>
+        <visual>
+            <origin xyz="0 0 0" rpy="0 0 0"/>
+            <geometry>
+                <mesh filename="package://robot_launcher_cpp/meshes/wheel.stl" scale="0.01 0.01 0.01"/>
+            </geometry>
+            <material name="red"/>
+        </visual>
+        <collision>
+            <origin xyz="0 0 0" rpy="0 0 0"/>
+            <geometry>
+                <mesh filename="package://robot_launcher_cpp/meshes/wheel.stl" scale="0.01 0.01 0.01"/>
+            </geometry>
+        </collision>
+    </link>
+    <link name="wheelfr_link">
+        <inertial>
+            <origin xyz="0 0 0" rpy="0 0 0"/>
+            <mass value="0.303"/>
+            <inertia ixx="2.05e-04" iyy="2.05e-04" izz="3.79e-04" ixy="0" ixz="0" iyz="0"/>
+        </inertial>
+        <visual>
+            <origin xyz="0 0 0" rpy="0 0 0"/>
+            <geometry>
+                <mesh filename="package://robot_launcher_cpp/meshes/wheel.stl" scale="0.01 0.01 0.01"/>
+            </geometry>
+            <material name="red"/>
+        </visual>
+        <collision>
+            <origin xyz="0 0 0" rpy="0 0 0"/>
+            <geometry>
+                <mesh filename="package://robot_launcher_cpp/meshes/wheel.stl" scale="0.01 0.01 0.01"/>
+            </geometry>
+        </collision>
+    </link>
+    <link name="wheelbl_link">
+        <inertial>
+            <origin xyz="0 0 0" rpy="0 0 0"/>
+            <mass value="0.303"/>
+            <inertia ixx="2.05e-04" iyy="2.05e-04" izz="3.79e-04" ixy="0" ixz="0" iyz="0"/>
+        </inertial>
+        <visual>
+            <origin xyz="0 0 0" rpy="0 0 0"/>
+            <geometry>
+                <mesh filename="package://robot_launcher_cpp/meshes/wheel.stl" scale="0.01 0.01 0.01"/>
+            </geometry>
+            <material name="yellow"/>
+        </visual>
+        <collision>
+            <origin xyz="0 0 0" rpy="0 0 0"/>
+            <geometry>
+                <mesh filename="package://robot_launcher_cpp/meshes/wheel.stl" scale="0.01 0.01 0.01"/>
+            </geometry>
+        </collision>
+    </link>
+    <link name="wheelbr_link">
+        <inertial>
+            <origin xyz="0 0 0" rpy="0 0 0"/>
+            <mass value="0.303"/>
+            <inertia ixx="2.05e-04" iyy="2.05e-04" izz="3.79e-04" ixy="0" ixz="0" iyz="0"/>
+        </inertial>
+        <visual>
+            <origin xyz="0 0 0" rpy="0 0 0"/>
+            <geometry>
+                <mesh filename="package://robot_launcher_cpp/meshes/wheel.stl" scale="0.01 0.01 0.01"/>
+            </geometry>
+            <material name="yellow"/>
+        </visual>
+        <collision>
+            <origin xyz="0 0 0" rpy="0 0 0"/>
+            <geometry>
+                <mesh filename="package://robot_launcher_cpp/meshes/wheel.stl" scale="0.01 0.01 0.01"/>
+            </geometry>
+        </collision>
+    </link>
+    <link name="camera_link">
+        <inertial>
+            <origin xyz="0 0 0" rpy="0 0 0"/>
+            <mass value="0.116"/>
+            <inertia ixx="1.03e-04" iyy="1.47e-05" izz="1.05e-04" ixy="0" ixz="0" iyz="0"/>
+        </inertial>
+        <visual>
+            <origin xyz="0 0 0" rpy="0 0 0"/>
+            <geometry>
+                <mesh filename="package://robot_launcher_cpp/meshes/camera.stl" scale="0.01 0.01 0.01"/>
+            </geometry>
+            <material name="blue"/>
+        </visual>
+        <collision>
+            <origin xyz="0 0 0" rpy="0 0 0"/>
+            <geometry>
+                <mesh filename="package://robot_launcher_cpp/meshes/camera.stl" scale="0.01 0.01 0.01"/>
+            </geometry>
+        </collision>
+    </link>
+    <link name="camera_color_link"/>
+    <link name="base_scan">
+        <inertial>
+            <origin xyz="0 0 0" rpy="0 0 0"/>
+            <mass value="0.232"/>
+            <inertia ixx="1.102e-04" iyy="1.102e-04" izz="1.856e-04" ixy="0" ixz="0" iyz="0"/>
+        </inertial>
+        <visual>
+            <origin xyz="0 0 0" rpy="0 0 0"/>
+            <geometry>
+                <mesh filename="package://robot_launcher_cpp/meshes/lidar.stl" scale="0.01 0.01 0.01"/>
+            </geometry>
+            <material name="green"/>
+        </visual>
+        <collision>
+            <origin xyz="0 0 0" rpy="0 0 0"/>
+            <geometry>
+                <mesh filename="package://robot_launcher_cpp/meshes/lidar.stl" scale="0.01 0.01 0.01"/>
+            </geometry>
+        </collision>
+    </link>
+    <link name="imu_link">
+    </link>
+<!--JOINTS-->
+    <joint name="base_joint" type="fixed">
         <origin xyz="0 0 0.0875" rpy="0 0 0"/>
-        <mass value="6.935"/>
-        <inertia ixx="0.026" iyy="0.055" izz="0.075" ixy="0" ixz="0" iyz="0"/>
-    </inertial>
-    <visual>
-        <origin xyz="0 0 0.0875" rpy="0 0 0"/>
-        <geometry>
-            <mesh filename="package://robot_launcher_cpp/meshes/base_link.stl" scale="0.01 0.01 0.01"/>
-        </geometry>
-        <material name="white"/>
-    </visual>
-    <collision>
-        <origin xyz="0 0 0.0875" rpy="0 0 0"/>
-        <geometry>
-            <mesh filename="package://robot_launcher_cpp/meshes/base_link.stl" scale="0.01 0.01 0.01"/>
-        </geometry>
-    </collision>
-</link>
-<joint name="wheell_joint" type="continuous">
-    <origin xyz="-0.1 0.1125 0.05" rpy="1.571 0 0"/>
-    <parent link="base_link"/>
-    <child link="wheell_link"/>
-    <axis xyz="0 0 1"/>
-</joint>
-<link name="wheell_link">
-    <inertial>
-        <origin xyz="0 0 0" rpy="0 0 0"/>
-        <mass value="0.303"/>
-        <inertia ixx="2.05e-04" iyy="2.05e-04" izz="7.58e-04" ixy="0" ixz="0" iyz="0"/>
-    </inertial>
-    <visual>
-        <origin xyz="0 0 0" rpy="0 0 0"/>
-        <geometry>
-            <mesh filename="package://robot_launcher_cpp/meshes/wheel.stl" scale="0.01 0.01 0.01"/>
-        </geometry>
-        <material name="red"/>
-    </visual>
-    <collision>
-        <origin xyz="0 0 0" rpy="0 0 0"/>
-        <geometry>
-            <mesh filename="package://robot_launcher_cpp/meshes/wheel.stl" scale="0.01 0.01 0.01"/>
-        </geometry>
-    </collision>
-</link>
-<joint name="wheelr_joint" type="continuous">
-    <origin xyz="-0.1 -0.1125 0.05" rpy="1.571 0 0"/>
-    <parent link="base_link"/>
-    <child link="wheelr_link"/>
-    <axis xyz="0 0 1"/>
-</joint>
-<link name="wheelr_link">
-    <inertial>
-        <origin xyz="0 0 0" rpy="0 0 0"/>
-        <mass value="0.303"/>
-        <inertia ixx="2.05e-04" iyy="2.05e-04" izz="7.58e-04" ixy="0" ixz="0" iyz="0"/>
-    </inertial>
-    <visual>
-        <origin xyz="0 0 0" rpy="0 0 0"/>
-        <geometry>
-            <mesh filename="package://robot_launcher_cpp/meshes/wheel.stl" scale="0.01 0.01 0.01"/>
-        </geometry>
-        <material name="red"/>
-    </visual>
-    <collision>
-        <origin xyz="0 0 0" rpy="0 0 0"/>
-        <geometry>
-            <mesh filename="package://robot_launcher_cpp/meshes/wheel.stl" scale="0.01 0.01 0.01"/>
-        </geometry>
-    </collision>
-</link>
-<joint name="wheeldl_joint" type="continuous">
-    <origin xyz="0.1 0.1125 0.05" rpy="-1.571 0 0"/>
-    <parent link="base_link"/>
-    <child link="wheeldl_link"/>
-    <axis xyz="0 0 1"/>
-</joint>
-<link name="wheeldl_link">
-    <inertial>
-        <origin xyz="0 0 0" rpy="0 0 0"/>
-        <mass value="0.303"/>
-        <inertia ixx="2.05e-04" iyy="2.05e-04" izz="7.58e-04" ixy="0" ixz="0" iyz="0"/>
-    </inertial>
-    <visual>
-        <origin xyz="0 0 0" rpy="0 0 0"/>
-        <geometry>
-            <mesh filename="package://robot_launcher_cpp/meshes/wheel.stl" scale="0.01 0.01 0.01"/>
-        </geometry>
-        <material name="red"/>
-    </visual>
-    <collision>
-        <origin xyz="0 0 0" rpy="0 0 0"/>
-        <geometry>
-            <mesh filename="package://robot_launcher_cpp/meshes/wheel.stl" scale="0.01 0.01 0.01"/>
-        </geometry>
-    </collision>
-</link>
-<joint name="wheeldr_joint" type="continuous">
-    <origin xyz="0.1 -0.1125 0.05" rpy="-1.571 0 0"/>
-    <parent link="base_link"/>
-    <child link="wheeldr_link"/>
-    <axis xyz="0 0 1"/>
-</joint>
-<link name="wheeldr_link">
-    <inertial>
-        <origin xyz="0 0 0" rpy="0 0 0"/>
-        <mass value="0.303"/>
-        <inertia ixx="2.05e-04" iyy="2.05e-04" izz="7.58e-04" ixy="0" ixz="0" iyz="0"/>
-    </inertial>
-    <visual>
-        <origin xyz="0 0 0" rpy="0 0 0"/>
-        <geometry>
-            <mesh filename="package://robot_launcher_cpp/meshes/wheel.stl" scale="0.01 0.01 0.01"/>
-        </geometry>
-        <material name="red"/>
-    </visual>
-    <collision>
-        <origin xyz="0 0 0" rpy="0 0 0"/>
-        <geometry>
-            <mesh filename="package://robot_launcher_cpp/meshes/wheel.stl" scale="0.01 0.01 0.01"/>
-        </geometry>
-    </collision>
-</link>
-<joint name="camera_joint" type="fixed">
-    <origin xyz="0.165 0 0.0875" rpy="0 0 0"/>
-    <parent link="base_link"/>
-    <child link="camera_link"/>
-</joint>
-<link name="camera_link">
-    <inertial>
-        <origin xyz="0 0 0" rpy="0 0 0"/>
-        <mass value="0.116"/>
-        <inertia ixx="1.47e-05" iyy="1.03e-04" izz="1.05e-04" ixy="0" ixz="0" iyz="0"/>
-    </inertial>
-    <visual>
-        <origin xyz="0 0 0" rpy="0 0 0"/>
-        <geometry>
-            <mesh filename="package://robot_launcher_cpp/meshes/camera.stl" scale="0.01 0.01 0.01"/>
-        </geometry>
-        <material name="blue"/>
-    </visual>
-    <collision>
-        <origin xyz="0 0 0" rpy="0 0 0"/>
-        <geometry>
-            <mesh filename="package://robot_launcher_cpp/meshes/camera.stl" scale="0.01 0.01 0.01"/>
-        </geometry>
-    </collision>
-</link>
-<joint name="camera_optical_joint" type="fixed">
-    <origin xyz="0.015 0 0" rpy="0 1.57 0"/>
-    <parent link="camera_link"/>
-    <child link="camera_color_link"/>
-</joint>
-<link name="camera_color_link"/>
-<joint name="lidar_joint" type="fixed">
-    <origin xyz="0.1 0 0.14" rpy="0 0 0"/>
-    <parent link="base_link"/>
-    <child link="base_scan"/>
-</joint>
-<link name="base_scan">
-    <inertial>
-        <origin xyz="0 0 0" rpy="0 0 0"/>
-        <mass value="0.232"/>
-        <inertia ixx="1.1e-04" iyy="1.1e-04" izz="3.09e-05" ixy="0" ixz="0" iyz="0"/>
-    </inertial>
-    <visual>
-        <origin xyz="0 0 0" rpy="0 0 0"/>
-        <geometry>
-            <mesh filename="package://robot_launcher_cpp/meshes/lidar.stl" scale="0.01 0.01 0.01"/>
-        </geometry>
-        <material name="green"/>
-    </visual>
-    <collision>
-        <origin xyz="0 0 0" rpy="0 0 0"/>
-        <geometry>
-            <mesh filename="package://robot_launcher_cpp/meshes/lidar.stl" scale="0.01 0.01 0.01"/>
-        </geometry>
-    </collision>
-</link>
-<joint name="imu_joint" type="fixed">
-    <origin xyz="0 0 0.0875" rpy="0 0 0"/>
-    <parent link="base_link"/>
-    <child link="imu_link"/>
-</joint>
-<link name="imu_link">
-</link>
-<xacro:include filename="wrv3.gazebo"/>
+        <parent link="base_footprint"/>
+        <child link="base_link"/>
+    </joint>
+    <joint name="wheelfl_joint" type="continuous">
+        <origin xyz="0.1 0.1125 -0.0375" rpy="-1.571 0 0"/>
+        <parent link="base_link"/>
+        <child link="wheelfl_link"/>
+        <axis xyz="0 0 1"/>
+    </joint>
+    <joint name="wheelfr_joint" type="continuous">
+        <origin xyz="0.1 -0.1125 -0.0375" rpy="-1.571 0 0"/>
+        <parent link="base_link"/>
+        <child link="wheelfr_link"/>
+        <axis xyz="0 0 1"/>
+    </joint>
+    <joint name="wheelbl_joint" type="continuous">
+        <origin xyz="-0.1 0.1125 -0.0375" rpy="1.571 0 0"/>
+        <parent link="base_link"/>
+        <child link="wheelbl_link"/>
+        <axis xyz="0 0 1"/>
+    </joint>
+    <joint name="wheelbr_joint" type="continuous">
+        <origin xyz="-0.1 -0.1125 -0.0375" rpy="1.571 0 0"/>
+        <parent link="base_link"/>
+        <child link="wheelbr_link"/>
+        <axis xyz="0 0 1"/>
+    </joint>
+    <joint name="camera_joint" type="fixed">
+        <origin xyz="0.165 0 0.0" rpy="0 0 0"/>
+        <parent link="base_link"/>
+        <child link="camera_link"/>
+    </joint>
+    <joint name="camera_optical_joint" type="fixed">
+        <origin xyz="0.015 0 0" rpy="0 0 0"/>
+        <parent link="camera_link"/>
+        <child link="camera_color_link"/>
+    </joint>
+    <joint name="lidar_joint" type="fixed">
+        <origin xyz="0.1 0 0.0525" rpy="0 0 0"/>
+        <parent link="base_link"/>
+        <child link="base_scan"/>
+    </joint>
+    <joint name="imu_joint" type="fixed">
+        <origin xyz="0 0 0.0" rpy="0 0 0"/>
+        <parent link="base_link"/>
+        <child link="imu_link"/>
+    </joint>
+    <xacro:include filename="wrv3.gazebo"/>
 </robot>
